Commit message: 10.28加手臂，换了模型

File: resources/robots/x1/urdf/x1.urdf (robot description, URDF)
Before this commit: robot x1, 58 links, 57 joints
Links:
- removed link lumber_pitch
- removed link lumber_roll
- removed link lumber_yaw
- added link lumbar_pitch, mass 8.8571074; visual mesh filename=../meshes/lumbar_pitch.STL
- added link lumbar_roll, mass 0.03412073; visual mesh filename=../meshes/lumbar_roll.STL
- added link lumbar_yaw, mass 0.36251906; visual mesh filename=../meshes/lumbar_yaw.STL
Joints:
- removed joint lumber_pitch_joint
- removed joint lumber_roll_joint
- removed joint lumber_yaw_joint
- added joint lumbar_pitch_joint: type fixed, parent lumbar_roll, child lumbar_pitch, origin xyz=0 0 0 rpy=0 1.5707963267949 0, axis 0 0 -1, limit lower=-3.14 upper=3.14 effort=0 velocity=0
- added joint lumbar_roll_joint: type fixed, parent lumbar_yaw, child lumbar_roll, origin xyz=0 0 0.0405 rpy=1.57079632679491 0 -1.5707963267949, axis 0 0 1, limit lower=-3.14 upper=3.14 effort=0 velocity=0
- added joint lumbar_yaw_joint: type fixed, parent base_link, child lumbar_yaw, origin xyz=0.00244999999994827 0 0.115534033809005 rpy=0 0 -4.54911392613975E-05, axis 0 0 1, limit lower=-3.14 upper=3.14 effort=0 velocity=0
- joint left_elbow_pitch_joint: limit lower=-3.14 upper=3.14 effort=0 velocity=0 -> lower=-3.14 upper=3.14 effort=80 velocity=10; type fixed -> revolute
- joint left_elbow_yaw_joint: origin xyz=0 0.116999999999998 0.0310000000000001 rpy=1.5707963267949  -1.5708 0 -> xyz=0 0.116999999999998 0.0310000000000001 rpy=1.5707963267949 -1.5708 0
- joint left_shoulder_pitch_joint: limit lower=-3.14 upper=3.14 effort=0 velocity=0 -> lower=-3.14 upper=3.14 effort=50 velocity=24; parent lumber_pitch -> lumbar_pitch; type fixed -> revolute
- joint left_shoulder_roll_joint: limit lower=-3.14 upper=3.14 effort=0 velocity=0 -> lower=-3.14 upper=3.14 effort=80 velocity=10; type fixed -> revolute
- joint right_elbow_pitch_joint: limit lower=-3.14 upper=3.14 effort=0 velocity=0 -> lower=-3.14 upper=3.14 effort=80 velocity=10; type fixed -> revolute
- joint right_shoulder_pitch_joint: limit lower=-3.14 upper=3.14 effort=0 velocity=0 -> lower=-3.14 upper=3.14 effort=50 velocity=24; parent lumber_pitch -> lumbar_pitch; type fixed -> revolute
- joint right_shoulder_roll_joint: limit lower=-3.14 upper=3.14 effort=0 velocity=0 -> lower=-3.14 upper=3.14 effort=80 velocity=10; type fixed -> revolute
- joint waist_motor_a_link_joint: parent lumber_pitch -> lumbar_pitch
- joint waist_motor_b_link_joint: parent lumber_pitch -> lumbar_pitch
